Commit message: movable swing arm

File: conveyorbelt_gazebo/models/swing_arm2/swing_arm2.urdf.xacro (robot description, xacro)
@@ -1,107 +1,108 @@
 <?xml version="1.0"?>
 <robot xmlns:xacro="http://www.ros.org/wiki/xacro" name="swing_arm2">
-    <link name="base_link">
-        <visual>
-            <geometry>
-                <box size="0.5 0.5 0.25"/>
-            </geometry>
-        </visual>
-        <collision>
-            <geometry>
-                <box size="0.5 0.5 0.25"/>
-            </geometry>
-        </collision>
-        <inertial>
-            <mass value="10000.0"/>
-            <inertia ixx="100.0" ixy="0" ixz="0" iyy="100.0" iyz="0" izz="100.0"/>
-        </inertial>
-    </link>
-    <link name="turret_link">
-        <visual>
-            <geometry>
-                <cylinder radius="0.02" length="0.65"/>
-            </geometry>
-        </visual>
-        <collision>
-            <geometry>
-                <cylinder radius="0.02" length="0.65"/>
-            </geometry>
-        </collision>
-        <inertial>
-            <mass value="1.0"/>
-            <inertia ixx="0.01" ixy="0" ixz="0" iyy="0.01" iyz="0" izz="0.01"/>
-        </inertial>
-    </link>
-    <link name="boom_link">
-        <visual>
-            <geometry>
-                <box size="0.015 0.3 0.05"/>
-            </geometry>
-        </visual>
-        <collision>
-            <geometry>
-                <box size="0.015 0.3 0.05"/>
-            </geometry>
-        </collision>
-        <inertial>
-            <mass value="0.5"/>
-            <inertia ixx="0.01" ixy="0" ixz="0" iyy="0.01" iyz="0" izz="0.01"/>
-        </inertial>
-    </link>
-    <link name="diverter_link">
-        <visual>
-            <geometry>
-                <box size="0.015 0.32 0.05"/>
-            </geometry>
-            <origin xyz="0 0 0" rpy="0 0 0"/>
-        </visual>
-        <collision>
-            <geometry>
-                <box size="0.015 0.32 0.05"/>
-            </geometry>
-            <origin xyz="0 0 0" rpy="0 0 0"/>
-        </collision>
-        <inertial>
-            <mass value="5"/>
-            <inertia ixx="0.1" ixy="0" ixz="0" iyy="0.1" iyz="0" izz="0.1"/>
-        </inertial>
-    </link>
-    <joint name='base_link_JOINT_0' type='fixed'>
-        <parent link="base_link"/>
-        <child link="turret_link"/>
-        <origin xyz="0 0 0.45" rpy="0 0 0"/>
+  <link name="base_link">
+    <visual>
+      <geometry>
+        <box size="0.5 0.5 0.25" />
+      </geometry>
+    </visual>
+    <collision>
+      <geometry>
+        <box size="0.5 0.5 0.25" />
+      </geometry>
+    </collision>
+    <inertial>
+      <mass value="10000.0" />
+      <inertia ixx="100.0" ixy="0" ixz="0" iyy="100.0" iyz="0" izz="100.0" />
+    </inertial>
+  </link>
+  <link name="turret_link">
+    <visual>
+      <geometry>
+        <cylinder radius="0.02" length="0.65" />
+      </geometry>
+    </visual>
+    <collision>
+      <geometry>
+        <cylinder radius="0.02" length="0.65" />
+      </geometry>
+    </collision>
+    <inertial>
+      <mass value="1.0" />
+      <inertia ixx="0.01" ixy="0" ixz="0" iyy="0.01" iyz="0" izz="0.01" />
+    </inertial>
+  </link>
+  <link name="boom_link">
+    <visual>
+      <geometry>
+        <box size="0.015 0.3 0.05" />
+      </geometry>
+    </visual>
+    <collision>
+      <geometry>
+        <box size="0.015 0.3 0.05" />
+      </geometry>
+    </collision>
+    <inertial>
+      <mass value="0.5" />
+      <inertia ixx="0.01" ixy="0" ixz="0" iyy="0.01" iyz="0" izz="0.01" />
+    </inertial>
+  </link>
+  <link name="diverter_link">
+    <visual>
+      <geometry>
+        <box size="0.015 0.32 0.05" />
+      </geometry>
+      <origin xyz="0 0 0" rpy="0 0 0" />
+    </visual>
+    <collision>
+      <geometry>
+        <box size="0.015 0.32 0.05" />
+      </geometry>
+      <origin xyz="0 0 0" rpy="0 0 0" />
+    </collision>
+    <inertial>
+      <mass value="5" />
+      <inertia ixx="0.1" ixy="0" ixz="0" iyy="0.1" iyz="0" izz="0.1" />
+    </inertial>
+  </link>
+  <joint name='base_link_JOINT_0' type='fixed'>
+    <parent link="base_link" />
+    <child link="turret_link" />
+    <origin xyz="0 0 0.45" rpy="0 0 0" />
+  </joint>
+  <joint name='turret_link_JOINT_0' type='fixed'>
+    <parent link="turret_link" />
+    <child link="boom_link" />
+    <origin xyz="0 0.15 0.25" rpy="0 0 0" />
+  </joint>
+  <joint name='boom_link_JOINT_0' type='revolute'>
+    <parent link="boom_link" />
+    <child link="diverter_link" />
+    <origin xyz="0 0.15 -0.05" rpy="0 0 0" />
+    <limit lower="-3.14159" upper="3.14159" effort="1000" velocity="10.0" />
+    <axis xyz="0 0 1" />
+    <dynamics damping="0" friction="0" />
+  </joint>
+  <ros2_control name="swing_arm_system" type="system">
+    <hardware>
+      <plugin>gazebo_ros2_control/GazeboSystem</plugin>
+    </hardware>
+    <joint name="boom_link_JOINT_0">
+      <command_interface name="effort">
+        <param name="min">-1000</param>
+        <param name="max">1000</param>
+      </command_interface>
+      <state_interface name="position" />
+      <state_interface name="velocity" />
+      <state_interface name="effort" />
     </joint>
-    <joint name='turret_link_JOINT_0' type='fixed'>
-        <parent link="turret_link"/>
-        <child link="boom_link"/>
-        <origin xyz="0 0.15 0.25" rpy="0 0 0"/>
-    </joint>
-    <joint name='boom_link_JOINT_0' type='revolute'>
-        <parent link="boom_link"/>
-        <child link="diverter_link"/>
-        <origin xyz="0 0.15 -0.05" rpy="0 0 0"/>
-        <limit lower="-3.14159" upper="3.14159" effort="1000" velocity="10.0"/>
-        <axis xyz="0 0 1"/>
-        <dynamics damping="0" friction="0"/>
-    </joint>
-<ros2_control name="swing_arm_system" type="system">
-  <hardware>
-    <plugin>gazebo_ros2_control/GazeboSystem</plugin>
-  </hardware>
-  <joint name="boom_link_JOINT_0">
-    <command_interface name="effort">
-      <param name="min">-1000</param>
-      <param name="max">1000</param>
-    </command_interface>
-    <state_interface name="position"/>
-    <state_interface name="velocity"/>
-    <state_interface name="effort"/>
-  </joint>
-</ros2_control>
-<gazebo>
-  <plugin filename="libgazebo_ros2_control.so" name="gazebo_ros2_control">
-    <!-- <parameters>/home/jacob/code/conveyor-gate/src/conveyor-model/conveyorbelt_gazebo/config/swing_arm_controllers.yaml</parameters> -->
-    <parameters>$(find conveyorbelt_gazebo)/config/swing_arm_controllers.yaml</parameters>
-  </plugin>
-</gazebo>
+  </ros2_control>
+  <gazebo>
+    <plugin filename="libgazebo_ros2_control.so" name="gazebo_ros2_control">
+      <!--
+      <parameters>/home/jacob/code/conveyor-gate/src/conveyor-model/conveyorbelt_gazebo/config/swing_arm_controllers.yaml</parameters> -->
+      <parameters>$(find conveyorbelt_gazebo)/config/swing_arm_controllers.yaml</parameters>
+    </plugin>
+  </gazebo>
 </robot>
